File: Split-MX-Hotswap/Split-MX-Hotswap.kicad_pcb (KiCad board)
At the start: 2 copper layers, 398 x 150.2 mm, 124 parts, among them J1 Conn_02x25_Counter_Clockwise, J2 Conn_02x25_Counter_Clockwise

Commit message: grounded board
Connections:
- J1 pad 19: unconnected-(J1-Pin_19-Pad19) -> GND
- J1 pad 39: unconnected-(J1-Pin_39-Pad39) -> GND
- J2 pad 19: unconnected-(J2-Pin_19-Pad19) -> GND
- J2 pad 39: unconnected-(J2-Pin_39-Pad39) -> GND
Routing:
- added copper zone on B.Cu, net GND
- added copper zone on F.Cu, net GND
Other:
- outline, holes or cut-outs redrawn
