File: Split-MX-Hotswap/Split-MX-Hotswap.kicad_sch (KiCad schematic)
At the start: 124 parts, among them J1 Conn_02x25_Counter_Clockwise, J2 Conn_02x25_Counter_Clockwise

Commit message: grounded board
Connections:
- net GND: now reaches J1.19 (Pin_19)
- net GND: now also J1.39 (Pin_39), J2.19 (Pin_19), J2.39 (Pin_39)
Changed lines of the file:
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@@
+		)
+	)
+	(global_label "GND"
+		(shape input)
+		(at 6.35 170.18 180)
+		(fields_autoplaced yes)
+		(effects
+			(font
+				(size 1.27 1.27)
+			)
+			(justify right)
+		)
+		(property "Intersheetrefs" "${INTERSHEET_REFS}"
+			(at -0.5057 170.18 0)
+			(effects
+				(font
+					(size 1.27 1.27)
+				)
+				(justify right)
+				(hide yes)
+			)
 		)
 	)
@@
 		)
 	)
+	(global_label "GND"
+		(shape input)
+		(at 114.3 191.77 180)
+		(fields_autoplaced yes)
+		(effects
+			(font
+				(size 1.27 1.27)
+			)
+			(justify right)
+		)
+		(property "Intersheetrefs" "${INTERSHEET_REFS}"
+			(at 107.4443 191.77 0)
+			(effects
+				(font
+					(size 1.27 1.27)
+				)
+				(justify right)
+				(hide yes)
+			)
+		)
+	)
 	(global_label "R2-L"
 		(shape input)
@@
 		)
 	)
+	(global_label "GND"
+		(shape input)
+		(at 127 173.99 0)
+		(fields_autoplaced yes)
+		(effects
+			(font
+				(size 1.27 1.27)
+			)
+			(justify left)
+		)
+		(property "Intersheetrefs" "${INTERSHEET_REFS}"
+			(at 133.8557 173.99 0)
+			(effects
+				(font
+					(size 1.27 1.27)
+				)
+				(justify left)
+				(hide yes)
+			)
+		)
+	)
 	(global_label "Row2-R"
 		(shape input)
@@
 				(hide yes)
 			)
+		)
+	)
+	(global_label "GND"
+		(shape input)
+		(at 19.05 152.4 0)
+		(fields_autoplaced yes)
+		(effects
+			(font
+				(size 1.27 1.27)
+			)
+			(justify left)
+		)
+		(property "Intersheetrefs" "${INTERSHEET_REFS}"
+			(at 25.9057 152.4 0)
+			(effects
+				(font
+					(size 1.27 1.27)
+				)
+				(justify left)
+				(hide yes)
+			)
